File: HT-manaita.kicad_pcb (KiCad board)
At the start: 2 copper layers, 0 parts

Commit message: 部品配置・基板外形作成
Parts:
- added D1: D, Diode_THT:D_A-405_P10.16mm_Horizontal, F.Cu at (253.9, 56.0)
- added D10: D, Diode_THT:D_A-405_P10.16mm_Horizontal, F.Cu at (234.9, 132.0)
- added D11: D, Diode_THT:D_A-405_P10.16mm_Horizontal, F.Cu at (215.8, 56.0)
- added D12: D, Diode_THT:D_A-405_P10.16mm_Horizontal, F.Cu at (215.8, 75.0)
- added D13: D, Diode_THT:D_A-405_P10.16mm_Horizontal, F.Cu at (215.9, 94.0)
- added D14: D, Diode_THT:D_A-405_P10.16mm_Horizontal, F.Cu at (215.8, 113.0)
- added D15: D, Diode_THT:D_A-405_P10.16mm_Horizontal, F.Cu at (215.8, 132.0)
- added D16: D, Diode_THT:D_A-405_P10.16mm_Horizontal, F.Cu at (196.8, 56.0)
- added D17: D, Diode_THT:D_A-405_P10.16mm_Horizontal, F.Cu at (196.8, 75.0)
- added D18: D, Diode_THT:D_A-405_P10.16mm_Horizontal, F.Cu at (196.8, 94.0)
- added D19: D, Diode_THT:D_A-405_P10.16mm_Horizontal, F.Cu at (196.8, 113.0)
- added D2: D, Diode_THT:D_A-405_P10.16mm_Horizontal, F.Cu at (253.8, 75.0)
- added D20: D, Diode_THT:D_A-405_P10.16mm_Horizontal, F.Cu at (196.8, 132.0)
- added D21: D, Diode_THT:D_A-405_P10.16mm_Horizontal, F.Cu at (177.8, 56.0)
- added D22: D, Diode_THT:D_A-405_P10.16mm_Horizontal, F.Cu at (177.8, 75.0)
- added D23: D, Diode_THT:D_A-405_P10.16mm_Horizontal, F.Cu at (177.8, 94.0)
- added D24: D, Diode_THT:D_A-405_P10.16mm_Horizontal, F.Cu at (177.8, 113.0)
- added D25: D, Diode_THT:D_A-405_P10.16mm_Horizontal, F.Cu at (177.8, 132.0)
- added D26: D, Diode_THT:D_A-405_P10.16mm_Horizontal, F.Cu at (158.9, 56.0)
- added D27: D, Diode_THT:D_A-405_P10.16mm_Horizontal, F.Cu at (158.8, 75.0)
- added D28: D, Diode_THT:D_A-405_P10.16mm_Horizontal, F.Cu at (158.9, 94.0)
- added D29: D, Diode_THT:D_A-405_P10.16mm_Horizontal, F.Cu at (158.8, 113.0)
- added D3: D, Diode_THT:D_A-405_P10.16mm_Horizontal, F.Cu at (253.8, 94.0)
- added D30: D, Diode_THT:D_A-405_P10.16mm_Horizontal, F.Cu at (158.8, 132.0)
- added D31: D, Diode_THT:D_A-405_P10.16mm_Horizontal, F.Cu at (129.7, 56.0)
- added D32: D, Diode_THT:D_A-405_P10.16mm_Horizontal, F.Cu at (129.7, 75.0)
- added D33: D, Diode_THT:D_A-405_P10.16mm_Horizontal, F.Cu at (129.7, 94.0)
- added D34: D, Diode_THT:D_A-405_P10.16mm_Horizontal, F.Cu at (129.7, 113.0)
- added D35: D, Diode_THT:D_A-405_P10.16mm_Horizontal, F.Cu at (129.7, 132.0)
- added D36: D, Diode_THT:D_A-405_P10.16mm_Horizontal, F.Cu at (110.6, 56.0)
- added D37: D, Diode_THT:D_A-405_P10.16mm_Horizontal, F.Cu at (110.7, 75.0)
- added D38: D, Diode_THT:D_A-405_P10.16mm_Horizontal, F.Cu at (110.7, 94.0)
- added D39: D, Diode_THT:D_A-405_P10.16mm_Horizontal, F.Cu at (110.7, 113.0)
- added D4: D, Diode_THT:D_A-405_P10.16mm_Horizontal, F.Cu at (253.8, 113.0)
- added D40: D, Diode_THT:D_A-405_P10.16mm_Horizontal, F.Cu at (110.7, 132.0)
- added D41: D, Diode_THT:D_A-405_P10.16mm_Horizontal, F.Cu at (91.6, 56.0)
- added D42: D, Diode_THT:D_A-405_P10.16mm_Horizontal, F.Cu at (91.7, 75.0)
- added D43: D, Diode_THT:D_A-405_P10.16mm_Horizontal, F.Cu at (91.7, 94.0)
- added D44: D, Diode_THT:D_A-405_P10.16mm_Horizontal, F.Cu at (91.7, 113.0)
- added D45: D, Diode_THT:D_A-405_P10.16mm_Horizontal, F.Cu at (91.7, 132.0)
- added D46: D, Diode_THT:D_A-405_P10.16mm_Horizontal, F.Cu at (72.6, 56.0)
- added D47: D, Diode_THT:D_A-405_P10.16mm_Horizontal, F.Cu at (72.6, 75.0)
- added D48: D, Diode_THT:D_A-405_P10.16mm_Horizontal, F.Cu at (72.6, 94.0)
- added D49: D, Diode_THT:D_A-405_P10.16mm_Horizontal, F.Cu at (72.6, 113.0)
- added D5: D, Diode_THT:D_A-405_P10.16mm_Horizontal, F.Cu at (253.8, 132.0)
- added D50: D, Diode_THT:D_A-405_P10.16mm_Horizontal, F.Cu at (72.6, 132.0)
- added D51: D, Diode_THT:D_A-405_P10.16mm_Horizontal, F.Cu at (53.6, 56.0)
- added D52: D, Diode_THT:D_A-405_P10.16mm_Horizontal, F.Cu at (53.6, 75.0)
- added D53: D, Diode_THT:D_A-405_P10.16mm_Horizontal, F.Cu at (52.7, 94.0)
- added D54: D, Diode_THT:D_A-405_P10.16mm_Horizontal, F.Cu at (53.6, 113.0)
- added D55: D, Diode_THT:D_A-405_P10.16mm_Horizontal, F.Cu at (53.6, 132.0)
- added D56: D, Diode_THT:D_A-405_P10.16mm_Horizontal, F.Cu at (34.6, 56.0)
- added D57: D, Diode_THT:D_A-405_P10.16mm_Horizontal, F.Cu at (34.6, 75.0)
- added D58: D, Diode_THT:D_A-405_P10.16mm_Horizontal, F.Cu at (33.6, 94.0)
- added D59: D, Diode_THT:D_A-405_P10.16mm_Horizontal, F.Cu at (34.7, 113.0)
- added D6: D, Diode_THT:D_A-405_P10.16mm_Horizontal, F.Cu at (234.8, 56.0)
- added D60: D, Diode_THT:D_A-405_P10.16mm_Horizontal, F.Cu at (34.6, 132.0)
- added D7: D, Diode_THT:D_A-405_P10.16mm_Horizontal, F.Cu at (234.8, 75.0)
- added D8: D, Diode_THT:D_A-405_P10.16mm_Horizontal, F.Cu at (234.9, 94.0)
- added D9: D, Diode_THT:D_A-405_P10.16mm_Horizontal, F.Cu at (234.9, 113.0)
- added J1: Conn_01x12_Pin, Connector_PinHeader_2.54mm:PinHeader_1x12_P2.54mm_Vertical, F.Cu at (258.5, 55.1)
- added J2: Conn_01x12_Pin, Connector_PinHeader_2.54mm:PinHeader_1x12_P2.54mm_Vertical, F.Cu at (273.7, 55.1)
- added SW1: SW_Push, Button_Switch_Keyboard:SW_Cherry_MX_1.00u_PCB, F.Cu at (249.4, 59.6)
- added SW10: SW_Push, Button_Switch_Keyboard:SW_Cherry_MX_1.00u_PCB, F.Cu at (230.4, 135.7)
- added SW11: SW_Push, Button_Switch_Keyboard:SW_Cherry_MX_1.00u_PCB, F.Cu at (211.4, 59.6)
- added SW12: SW_Push, Button_Switch_Keyboard:SW_Cherry_MX_1.00u_PCB, F.Cu at (211.4, 78.7)
- added SW13: SW_Push, Button_Switch_Keyboard:SW_Cherry_MX_1.00u_PCB, F.Cu at (211.4, 97.7)
- added SW14: SW_Push, Button_Switch_Keyboard:SW_Cherry_MX_1.00u_PCB, F.Cu at (211.4, 116.7)
- added SW15: SW_Push, Button_Switch_Keyboard:SW_Cherry_MX_1.00u_PCB, F.Cu at (211.4, 135.7)
- added SW16: SW_Push, Button_Switch_Keyboard:SW_Cherry_MX_1.00u_PCB, F.Cu at (192.4, 59.6)
- added SW17: SW_Push, Button_Switch_Keyboard:SW_Cherry_MX_1.00u_PCB, F.Cu at (192.4, 78.7)
- added SW18: SW_Push, Button_Switch_Keyboard:SW_Cherry_MX_1.00u_PCB, F.Cu at (192.4, 97.7)
- added SW19: SW_Push, Button_Switch_Keyboard:SW_Cherry_MX_1.00u_PCB, F.Cu at (192.4, 116.7)
- added SW2: SW_Push, Button_Switch_Keyboard:SW_Cherry_MX_1.00u_PCB, F.Cu at (249.4, 78.7)
- added SW20: SW_Push, Button_Switch_Keyboard:SW_Cherry_MX_1.00u_PCB, F.Cu at (192.4, 135.7)
- added SW21: SW_Push, Button_Switch_Keyboard:SW_Cherry_MX_1.00u_PCB, F.Cu at (173.4, 59.6)
- added SW22: SW_Push, Button_Switch_Keyboard:SW_Cherry_MX_1.00u_PCB, F.Cu at (173.4, 78.7)
- added SW23: SW_Push, Button_Switch_Keyboard:SW_Cherry_MX_1.00u_PCB, F.Cu at (173.4, 97.7)
- added SW24: SW_Push, Button_Switch_Keyboard:SW_Cherry_MX_1.00u_PCB, F.Cu at (173.4, 116.7)
- added SW25: SW_Push, Button_Switch_Keyboard:SW_Cherry_MX_1.00u_PCB, F.Cu at (173.4, 135.7)
- added SW26: SW_Push, Button_Switch_Keyboard:SW_Cherry_MX_1.00u_PCB, F.Cu at (154.4, 59.6)
- added SW27: SW_Push, Button_Switch_Keyboard:SW_Cherry_MX_1.00u_PCB, F.Cu at (154.4, 78.7)
- added SW28: SW_Push, Button_Switch_Keyboard:SW_Cherry_MX_1.00u_PCB, F.Cu at (154.4, 97.7)
- added SW29: SW_Push, Button_Switch_Keyboard:SW_Cherry_MX_1.00u_PCB, F.Cu at (154.4, 116.7)
- added SW3: SW_Push, Button_Switch_Keyboard:SW_Cherry_MX_1.00u_PCB, F.Cu at (249.4, 97.7)
- added SW30: SW_Push, Button_Switch_Keyboard:SW_Cherry_MX_1.00u_PCB, F.Cu at (154.4, 135.7)
- added SW31: SW_Push, Button_Switch_Keyboard:SW_Cherry_MX_1.00u_PCB, F.Cu at (135.4, 59.6)
- added SW32: SW_Push, Button_Switch_Keyboard:SW_Cherry_MX_1.00u_PCB, F.Cu at (135.4, 78.7)
- added SW33: SW_Push, Button_Switch_Keyboard:SW_Cherry_MX_1.00u_PCB, F.Cu at (135.4, 97.7)
- added SW34: SW_Push, Button_Switch_Keyboard:SW_Cherry_MX_1.00u_PCB, F.Cu at (135.4, 116.7)
- added SW35: SW_Push, Button_Switch_Keyboard:SW_Cherry_MX_1.00u_PCB, F.Cu at (135.4, 135.7)
- added SW36: SW_Push, Button_Switch_Keyboard:SW_Cherry_MX_1.00u_PCB, F.Cu at (116.4, 59.6)
- added SW37: SW_Push, Button_Switch_Keyboard:SW_Cherry_MX_1.00u_PCB, F.Cu at (116.4, 78.7)
- added SW38: SW_Push, Button_Switch_Keyboard:SW_Cherry_MX_1.00u_PCB, F.Cu at (116.4, 97.7)
- added SW39: SW_Push, Button_Switch_Keyboard:SW_Cherry_MX_1.00u_PCB, F.Cu at (116.4, 116.7)
- added SW4: SW_Push, Button_Switch_Keyboard:SW_Cherry_MX_1.00u_PCB, F.Cu at (249.4, 116.7)
- added SW40: SW_Push, Button_Switch_Keyboard:SW_Cherry_MX_1.00u_PCB, F.Cu at (116.4, 135.7)
- added SW41: SW_Push, Button_Switch_Keyboard:SW_Cherry_MX_1.00u_PCB, F.Cu at (97.4, 59.6)
- added SW42: SW_Push, Button_Switch_Keyboard:SW_Cherry_MX_1.00u_PCB, F.Cu at (97.4, 78.7)
- added SW43: SW_Push, Button_Switch_Keyboard:SW_Cherry_MX_1.00u_PCB, F.Cu at (97.4, 97.7)
- added SW44: SW_Push, Button_Switch_Keyboard:SW_Cherry_MX_1.00u_PCB, F.Cu at (97.4, 116.7)
- added SW45: SW_Push, Button_Switch_Keyboard:SW_Cherry_MX_1.00u_PCB, F.Cu at (97.4, 135.7)
- added SW46: SW_Push, Button_Switch_Keyboard:SW_Cherry_MX_1.00u_PCB, F.Cu at (78.4, 59.6)
- added SW47: SW_Push, Button_Switch_Keyboard:SW_Cherry_MX_1.00u_PCB, F.Cu at (78.4, 78.7)
- added SW48: SW_Push, Button_Switch_Keyboard:SW_Cherry_MX_1.00u_PCB, F.Cu at (78.4, 97.7)
- added SW49: SW_Push, Button_Switch_Keyboard:SW_Cherry_MX_1.00u_PCB, F.Cu at (78.4, 116.7)
- added SW5: SW_Push, Button_Switch_Keyboard:SW_Cherry_MX_1.00u_PCB, F.Cu at (249.4, 135.7)
- added SW50: SW_Push, Button_Switch_Keyboard:SW_Cherry_MX_1.00u_PCB, F.Cu at (78.4, 135.7)
- added SW51: SW_Push, Button_Switch_Keyboard:SW_Cherry_MX_1.00u_PCB, F.Cu at (59.4, 59.6)
- added SW52: SW_Push, Button_Switch_Keyboard:SW_Cherry_MX_1.00u_PCB, F.Cu at (59.4, 78.7)
- added SW53: SW_Push, Button_Switch_Keyboard:SW_Cherry_MX_1.00u_PCB, F.Cu at (59.4, 97.7)
- added SW54: SW_Push, Button_Switch_Keyboard:SW_Cherry_MX_1.00u_PCB, F.Cu at (59.4, 116.7)
- added SW55: SW_Push, Button_Switch_Keyboard:SW_Cherry_MX_1.00u_PCB, F.Cu at (59.4, 135.7)
- added SW56: SW_Push, Button_Switch_Keyboard:SW_Cherry_MX_1.00u_PCB, F.Cu at (40.4, 59.6)
- added SW57: SW_Push, Button_Switch_Keyboard:SW_Cherry_MX_1.00u_PCB, F.Cu at (40.4, 78.7)
- added SW58: SW_Push, Button_Switch_Keyboard:SW_Cherry_MX_1.00u_PCB, F.Cu at (40.4, 97.7)
- added SW59: SW_Push, Button_Switch_Keyboard:SW_Cherry_MX_1.00u_PCB, F.Cu at (40.4, 116.7)
- added SW6: SW_Push, Button_Switch_Keyboard:SW_Cherry_MX_1.00u_PCB, F.Cu at (230.4, 59.6)
- added SW60: SW_Push, Button_Switch_Keyboard:SW_Cherry_MX_1.00u_PCB, F.Cu at (40.4, 135.7)
- added SW7: SW_Push, Button_Switch_Keyboard:SW_Cherry_MX_1.00u_PCB, F.Cu at (230.4, 78.7)
- added SW8: SW_Push, Button_Switch_Keyboard:SW_Cherry_MX_1.00u_PCB, F.Cu at (230.4, 97.7)
- added SW9: SW_Push, Button_Switch_Keyboard:SW_Cherry_MX_1.00u_PCB, F.Cu at (230.4, 116.7)
Routing:
- net unconnected-(SW56-Pad1): track 0.00 -> 76.0 mm
- net unconnected-(SW51-Pad1): track 0.00 -> 76.0 mm
- net unconnected-(SW46-Pad1): track 0.00 -> 76.0 mm
- net unconnected-(SW41-Pad1): track 0.00 -> 76.0 mm
- net unconnected-(SW36-Pad1): track 0.00 -> 76.0 mm
- net unconnected-(SW31-Pad1): track 0.00 -> 76.0 mm
- net unconnected-(SW26-Pad1): track 0.00 -> 76.0 mm
- net ROW4: track 0.00 -> 76.0 mm
- net ROW3: track 0.00 -> 76.0 mm
- net ROW2: track 0.00 -> 76.0 mm
- net ROW1: track 0.00 -> 76.0 mm
- net ROW0: track 0.00 -> 76.0 mm
- net Net-(D1-A): track 0.00 -> 6.48 mm
- net Net-(D56-K): track 0.00 -> 6.48 mm
- net Net-(D51-K): track 0.00 -> 6.48 mm
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Other:
- board outline added: 248.9 x 99.1 mm
