File: HT-manaita.kicad_pcb (KiCad board)
At the start: 2 copper layers, 248.9 x 99.1 mm, 122 parts, among them J1 Conn_01x12_Pin, J2 Conn_01x12_Pin, SW1 SW_Push, SW10 SW_Push, SW11 SW_Push, SW12 SW_Push, SW13 SW_Push, SW14 SW_Push, SW15 SW_Push, SW16 SW_Push, SW17 SW_Push, SW18 SW_Push, SW19 SW_Push, SW2 SW_Push, SW20 SW_Push, SW21 SW_Push, SW22 SW_Push, SW23 SW_Push, SW24 SW_Push, SW25 SW_Push, SW26 SW_Push, SW27 SW_Push, SW28 SW_Push, SW29 SW_Push, SW3 SW_Push, SW30 SW_Push, SW31 SW_Push, SW32 SW_Push, SW33 SW_Push, SW34 SW_Push, SW35 SW_Push, SW36 SW_Push, SW37 SW_Push, SW38 SW_Push, SW39 SW_Push, SW4 SW_Push, SW40 SW_Push, SW41 SW_Push, SW42 SW_Push, SW43 SW_Push, SW44 SW_Push, SW45 SW_Push, SW46 SW_Push, SW47 SW_Push, SW48 SW_Push, SW49 SW_Push, SW5 SW_Push, SW50 SW_Push, SW51 SW_Push, SW52 SW_Push, SW53 SW_Push, SW54 SW_Push, SW55 SW_Push, SW56 SW_Push, SW57 SW_Push, SW58 SW_Push, SW59 SW_Push, SW6 SW_Push, SW60 SW_Push, SW7 SW_Push, SW8 SW_Push, SW9 SW_Push

Commit message: HT-manaita_v1.0 基板作成
Parts:
- moved D15 0.80 mm to (215.0, 132.0)
- moved D20 0.80 mm to (196.0, 132.0)
- moved D25 0.80 mm to (177.0, 132.0)
- moved D30 0.80 mm to (158.0, 132.0)
- moved D35 0.80 mm to (128.9, 132.0)
- moved D5 0.80 mm to (253.0, 132.0)
- moved D11 0.80 mm to (215.0, 56.0)
- moved D16 0.80 mm to (196.0, 56.0)
- moved D21 0.80 mm to (177.0, 56.0)
- moved D31 0.80 mm to (128.9, 56.0)
- moved D6 0.80 mm to (234.0, 56.0)
- moved J1 0.80 mm to (257.7, 55.1)
- moved J2 0.80 mm to (272.9, 55.1)
- moved D12 0.80 mm to (215.0, 75.0)
- moved D14 0.80 mm to (215.0, 113.0)
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Connections:
- D1 pad 1: COL0 -> COL4
- D10 pad 1: COL0 -> COL1
- D11 pad 1: COL0 -> COL1
- D13 pad 1: COL0 -> COL4
- D14 pad 1: COL0 -> COL3
- D15 pad 1: COL0 -> COL2
- D16 pad 1: COL0 -> COL2
- D17 pad 1: COL0 -> COL1
- D19 pad 1: COL0 -> COL4
- D19 pad 2: Net-(D19-A) -> unconnected-(D19-A-Pad2)
- D2 pad 1: COL0 -> COL3
- D20 pad 1: COL0 -> COL3
- D21 pad 1: COL0 -> COL3
- D22 pad 1: COL0 -> COL2
- D23 pad 1: COL0 -> COL1
- D25 pad 1: COL0 -> COL4
- D26 pad 1: COL0 -> COL4
- D27 pad 1: COL0 -> COL3
- D28 pad 1: COL0 -> COL2
- D29 pad 1: COL0 -> COL1
- D3 pad 1: COL0 -> COL2
- D32 pad 2: COL0 -> COL4
- D33 pad 2: COL0 -> COL3
- D34 pad 2: COL0 -> COL2
- D35 pad 2: COL0 -> COL1
- D36 pad 2: COL0 -> COL1
- D38 pad 2: COL0 -> COL4
- D39 pad 2: COL0 -> COL3
- D4 pad 1: COL0 -> COL1
- D40 pad 2: COL0 -> COL2
- D41 pad 2: COL0 -> COL2
- D42 pad 2: COL0 -> COL1
- D44 pad 2: COL0 -> COL4
- D45 pad 2: COL0 -> COL3
- D46 pad 2: COL0 -> COL3
- D47 pad 2: COL0 -> COL2
- D48 pad 2: COL0 -> COL1
- D50 pad 2: COL0 -> COL4
- D51 pad 2: COL0 -> COL4
- D52 pad 2: COL0 -> COL3
- D53 pad 2: COL0 -> COL2
- D54 pad 2: COL0 -> COL1
- D57 pad 2: COL0 -> COL4
- D58 pad 2: COL0 -> COL3
- D59 pad 2: COL0 -> COL2
- D60 pad 2: COL0 -> COL1
- D7 pad 1: COL0 -> COL4
- D8 pad 1: COL0 -> COL3
- D9 pad 1: COL0 -> COL2
- J1 pad 10: COL0 -> COL2
- J1 pad 11: COL0 -> COL1
- J1 pad 3: GND -> unconnected-(J1-Pin_3-Pad3)
- J1 pad 4: GND -> unconnected-(J1-Pin_4-Pad4)
- J1 pad 8: COL0 -> COL4
- J1 pad 9: COL0 -> COL3
- J2 pad 2: GND -> unconnected-(J2-Pin_2-Pad2)
- SW26 pad 1: unconnected-(SW26-Pad1) -> Net-(SW26-Pad1)
- SW27 pad 1: unconnected-(SW26-Pad1) -> Net-(SW26-Pad1)
- SW28 pad 1: unconnected-(SW26-Pad1) -> Net-(SW26-Pad1)
- SW29 pad 1: unconnected-(SW26-Pad1) -> Net-(SW26-Pad1)
- SW30 pad 1: unconnected-(SW26-Pad1) -> Net-(SW26-Pad1)
- SW31 pad 1: unconnected-(SW31-Pad1) -> Net-(SW31-Pad1)
- SW32 pad 1: unconnected-(SW31-Pad1) -> Net-(SW31-Pad1)
- SW33 pad 1: unconnected-(SW31-Pad1) -> Net-(SW31-Pad1)
- SW34 pad 1: unconnected-(SW31-Pad1) -> Net-(SW31-Pad1)
- SW35 pad 1: unconnected-(SW31-Pad1) -> Net-(SW31-Pad1)
- SW36 pad 1: unconnected-(SW36-Pad1) -> Net-(SW36-Pad1)
- SW37 pad 1: unconnected-(SW36-Pad1) -> Net-(SW36-Pad1)
- SW38 pad 1: unconnected-(SW36-Pad1) -> Net-(SW36-Pad1)
- SW39 pad 1: unconnected-(SW36-Pad1) -> Net-(SW36-Pad1)
- SW40 pad 1: unconnected-(SW36-Pad1) -> Net-(SW36-Pad1)
- SW41 pad 1: unconnected-(SW41-Pad1) -> Net-(SW41-Pad1)
- SW42 pad 1: unconnected-(SW41-Pad1) -> Net-(SW41-Pad1)
- SW43 pad 1: unconnected-(SW41-Pad1) -> Net-(SW41-Pad1)
- SW44 pad 1: unconnected-(SW41-Pad1) -> Net-(SW41-Pad1)
- SW45 pad 1: unconnected-(SW41-Pad1) -> Net-(SW41-Pad1)
- SW46 pad 1: unconnected-(SW46-Pad1) -> Net-(SW46-Pad1)
- SW47 pad 1: unconnected-(SW46-Pad1) -> Net-(SW46-Pad1)
- SW48 pad 1: unconnected-(SW46-Pad1) -> Net-(SW46-Pad1)
- SW49 pad 1: unconnected-(SW46-Pad1) -> Net-(SW46-Pad1)
- SW50 pad 1: unconnected-(SW46-Pad1) -> Net-(SW46-Pad1)
- SW51 pad 1: unconnected-(SW51-Pad1) -> Net-(SW51-Pad1)
- SW52 pad 1: unconnected-(SW51-Pad1) -> Net-(SW51-Pad1)
- SW53 pad 1: unconnected-(SW51-Pad1) -> Net-(SW51-Pad1)
- SW54 pad 1: unconnected-(SW51-Pad1) -> Net-(SW51-Pad1)
- SW55 pad 1: unconnected-(SW51-Pad1) -> Net-(SW51-Pad1)
- SW56 pad 1: unconnected-(SW56-Pad1) -> Net-(SW56-Pad1)
- SW57 pad 1: unconnected-(SW56-Pad1) -> Net-(SW56-Pad1)
- SW58 pad 1: unconnected-(SW56-Pad1) -> Net-(SW56-Pad1)
- SW59 pad 1: unconnected-(SW56-Pad1) -> Net-(SW56-Pad1)
- SW60 pad 1: unconnected-(SW56-Pad1) -> Net-(SW56-Pad1)
Routing:
- net COL0: track 0.00 -> 687.6 mm
- net COL1: track 0.00 -> 553.6 mm
- net COL4: track 0.00 -> 537.7 mm
- net COL2: track 0.00 -> 537.2 mm
- net COL3: track 0.00 -> 523.8 mm
- net ROW3: track 76.0 -> 194.5 mm
- net ROW2: track 76.0 -> 171.0 mm
- net unconnected-(SW56-Pad1): track 76.0 -> 0.00 mm
- net unconnected-(SW51-Pad1): track 76.0 -> 0.00 mm
- net unconnected-(SW46-Pad1): track 76.0 -> 0.00 mm
- net unconnected-(SW41-Pad1): track 76.0 -> 0.00 mm
- net unconnected-(SW36-Pad1): track 76.0 -> 0.00 mm
- net unconnected-(SW31-Pad1): track 76.0 -> 0.00 mm
- net unconnected-(SW26-Pad1): track 76.0 -> 0.00 mm
- net Net-(SW56-Pad1): track 0.00 -> 76.0 mm
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Other:
- board size 248.9 x 99.1 mm -> 251 x 101 mm
- board text added: "HT-manaita"
