File: HT-manaita.kicad_pcb (KiCad board)
At the start: 2 copper layers, 251 x 101 mm, 122 parts, among them J1 Conn_01x12_Pin, J2 Conn_01x12_Pin, SW1 SW_Push, SW10 SW_Push, SW11 SW_Push, SW12 SW_Push, SW13 SW_Push, SW14 SW_Push, SW15 SW_Push, SW16 SW_Push, SW17 SW_Push, SW18 SW_Push, SW19 SW_Push, SW2 SW_Push, SW20 SW_Push, SW21 SW_Push, SW22 SW_Push, SW23 SW_Push, SW24 SW_Push, SW25 SW_Push, SW26 SW_Push, SW27 SW_Push, SW28 SW_Push, SW29 SW_Push, SW3 SW_Push, SW30 SW_Push, SW31 SW_Push, SW32 SW_Push, SW33 SW_Push, SW34 SW_Push, SW35 SW_Push, SW36 SW_Push, SW37 SW_Push, SW38 SW_Push, SW39 SW_Push, SW4 SW_Push, SW40 SW_Push, SW41 SW_Push, SW42 SW_Push, SW43 SW_Push, SW44 SW_Push, SW45 SW_Push, SW46 SW_Push, SW47 SW_Push, SW48 SW_Push, SW49 SW_Push, SW5 SW_Push, SW50 SW_Push, SW51 SW_Push, SW52 SW_Push, SW53 SW_Push, SW54 SW_Push, SW55 SW_Push, SW56 SW_Push, SW57 SW_Push, SW58 SW_Push, SW59 SW_Push, SW6 SW_Push, SW60 SW_Push, SW7 SW_Push, SW8 SW_Push, SW9 SW_Push

Commit message: v2.0 アップデート
Parts:
- moved D13 1.26 mm to (213.9, 93.5)
- moved D28 1.26 mm to (156.9, 93.5)
- moved D8 1.26 mm to (232.9, 93.5)
- moved D9 1.26 mm to (232.9, 112.5)
- moved J2 1.26 mm to (271.8, 54.6)
- moved D1 1.26 mm to (251.9, 55.5)
- moved D26 1.26 mm to (156.9, 55.5)
- moved D10 1.26 mm to (232.9, 131.5)
- moved SW36 1.26 mm to (114.5, 59.2)
- moved SW37 1.26 mm to (114.5, 78.2)
- moved SW38 1.26 mm to (114.5, 97.2)
- moved SW39 1.26 mm to (114.5, 116.2)
- moved SW41 1.26 mm to (95.5, 59.2)
- moved SW42 1.26 mm to (95.5, 78.2)
- moved SW43 1.26 mm to (95.5, 97.2)
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Connections:
- D1 pad 1: COL4 -> ROW4
- D10 pad 1: COL1 -> ROW1
- D11 pad 1: COL1 -> ROW1
- D12 pad 1: COL0 -> ROW0
- D13 pad 1: COL4 -> ROW4
- D14 pad 1: COL3 -> ROW3
- D15 pad 1: COL2 -> ROW2
- D16 pad 1: COL2 -> ROW2
- D17 pad 1: COL1 -> ROW1
- D18 pad 1: COL0 -> ROW0
- D19 pad 1: COL4 -> ROW4
- D2 pad 1: COL3 -> ROW3
- D20 pad 1: COL3 -> ROW3
- D21 pad 1: COL3 -> ROW3
- D22 pad 1: COL2 -> ROW2
- D23 pad 1: COL1 -> ROW1
- D24 pad 1: COL0 -> ROW0
- D25 pad 1: COL4 -> ROW4
- D26 pad 1: COL4 -> ROW4
- D27 pad 1: COL3 -> ROW3
- D28 pad 1: COL2 -> ROW2
- D29 pad 1: COL1 -> ROW1
- D3 pad 1: COL2 -> ROW2
- D30 pad 1: COL0 -> ROW0
- D31 pad 2: COL0 -> ROW0
- D32 pad 2: COL4 -> ROW4
- D33 pad 2: COL3 -> ROW3
- D34 pad 2: COL2 -> ROW2
- D35 pad 2: COL1 -> ROW1
- D36 pad 2: COL1 -> ROW1
- D37 pad 2: COL0 -> ROW0
- D38 pad 2: COL4 -> ROW4
- D39 pad 2: COL3 -> ROW3
- D4 pad 1: COL1 -> ROW1
- D40 pad 2: COL2 -> ROW2
- D41 pad 2: COL2 -> ROW2
- D42 pad 2: COL1 -> ROW1
- D43 pad 2: COL0 -> ROW0
- D44 pad 2: COL4 -> ROW4
- D45 pad 2: COL3 -> ROW3
- D46 pad 2: COL3 -> ROW3
- D47 pad 2: COL2 -> ROW2
- D48 pad 2: COL1 -> ROW1
- D49 pad 2: COL0 -> ROW0
- D5 pad 1: COL0 -> ROW0
- D50 pad 2: COL4 -> ROW4
- D51 pad 2: COL4 -> ROW4
- D52 pad 2: COL3 -> ROW3
- D53 pad 2: COL2 -> ROW2
- D54 pad 2: COL1 -> ROW1
- D55 pad 2: COL0 -> ROW0
- D56 pad 2: COL0 -> ROW0
- D57 pad 2: COL4 -> ROW4
- D58 pad 2: COL3 -> ROW3
- D59 pad 2: COL2 -> ROW2
- D6 pad 1: COL0 -> ROW0
- D60 pad 2: COL1 -> ROW1
- D7 pad 1: COL4 -> ROW4
- D8 pad 1: COL3 -> ROW3
- D9 pad 1: COL2 -> ROW2
- J1 pad 7: COL0 -> COL5
- J2 pad 12: RW4 -> ROW4
- SW1 pad 1: ROW0 -> COL0
- SW10 pad 1: ROW1 -> COL1
- SW11 pad 1: ROW2 -> COL2
- SW12 pad 1: ROW2 -> COL2
- SW13 pad 1: ROW2 -> COL2
- SW14 pad 1: ROW2 -> COL2
- SW15 pad 1: ROW2 -> COL2
- SW16 pad 1: ROW3 -> COL3
- SW17 pad 1: ROW3 -> COL3
- SW18 pad 1: ROW3 -> COL3
- SW2 pad 1: ROW0 -> COL0
- SW20 pad 1: ROW3 -> COL3
- SW21 pad 1: ROW4 -> COL4
- SW22 pad 1: ROW4 -> COL4
- SW23 pad 1: ROW4 -> COL4
- SW24 pad 1: ROW4 -> COL4
- SW25 pad 1: ROW4 -> COL4
- SW26 pad 1: Net-(SW26-Pad1) -> COL5
- SW27 pad 1: Net-(SW26-Pad1) -> COL5
- SW28 pad 1: Net-(SW26-Pad1) -> COL5
- SW29 pad 1: Net-(SW26-Pad1) -> COL5
- SW3 pad 1: ROW0 -> COL0
- SW30 pad 1: Net-(SW26-Pad1) -> COL5
- SW31 pad 1: Net-(SW31-Pad1) -> COL0
- SW32 pad 1: Net-(SW31-Pad1) -> COL0
- SW33 pad 1: Net-(SW31-Pad1) -> COL0
- SW34 pad 1: Net-(SW31-Pad1) -> COL0
- SW35 pad 1: Net-(SW31-Pad1) -> COL0
- SW36 pad 1: Net-(SW36-Pad1) -> COL1
- SW37 pad 1: Net-(SW36-Pad1) -> COL1
- SW38 pad 1: Net-(SW36-Pad1) -> COL1
- SW39 pad 1: Net-(SW36-Pad1) -> COL1
- SW4 pad 1: ROW0 -> COL0
- SW40 pad 1: Net-(SW36-Pad1) -> COL1
- SW41 pad 1: Net-(SW41-Pad1) -> COL2
- SW42 pad 1: Net-(SW41-Pad1) -> COL2
- SW43 pad 1: Net-(SW41-Pad1) -> COL2
- SW44 pad 1: Net-(SW41-Pad1) -> COL2
- SW45 pad 1: Net-(SW41-Pad1) -> COL2
- SW46 pad 1: Net-(SW46-Pad1) -> COL3
- SW47 pad 1: Net-(SW46-Pad1) -> COL3
- SW48 pad 1: Net-(SW46-Pad1) -> COL3
- SW49 pad 1: Net-(SW46-Pad1) -> COL3
- SW5 pad 1: ROW0 -> COL0
- SW50 pad 1: Net-(SW46-Pad1) -> COL3
- SW51 pad 1: Net-(SW51-Pad1) -> COL4
- SW52 pad 1: Net-(SW51-Pad1) -> COL4
- SW53 pad 1: Net-(SW51-Pad1) -> COL4
- SW54 pad 1: Net-(SW51-Pad1) -> COL4
- SW55 pad 1: Net-(SW51-Pad1) -> COL4
- SW56 pad 1: Net-(SW56-Pad1) -> COL5
- SW57 pad 1: Net-(SW56-Pad1) -> COL5
- SW58 pad 1: Net-(SW56-Pad1) -> COL5
- SW59 pad 1: Net-(SW56-Pad1) -> COL5
- SW6 pad 1: ROW1 -> COL1
- SW60 pad 1: Net-(SW56-Pad1) -> COL5
- SW7 pad 1: ROW1 -> COL1
- SW8 pad 1: ROW1 -> COL1
- SW9 pad 1: ROW1 -> COL1
Routing:
- net ROW0: track 106.1 -> 659.9 mm, vias 0 -> 1
- net ROW3: track 194.5 -> 723.7 mm, vias 0 -> 1
- net ROW4: track 76.0 -> 567.3 mm, vias 0 -> 1
- net COL5: track 0.00 -> 488.3 mm, vias 0 -> 2
- net ROW1: track 147.8 -> 603.3 mm, vias 0 -> 1
- net ROW2: track 171.0 -> 625.9 mm, vias 0 -> 1
- net COL0: track 687.6 -> 352.9 mm, vias 0 -> 2
- net COL1: track 553.6 -> 380.5 mm, vias 0 -> 2
- net COL3: track 523.8 -> 358.7 mm, vias 0 -> 2
- net COL2: track 537.2 -> 406.8 mm, vias 0 -> 2
- net COL4: track 537.7 -> 461.0 mm, vias 0 -> 2
- net Net-(SW56-Pad1): track 76.0 -> 0.00 mm
- net Net-(SW51-Pad1): track 76.0 -> 0.00 mm
- net Net-(SW46-Pad1): track 76.0 -> 0.00 mm
- net Net-(SW41-Pad1): track 76.0 -> 0.00 mm
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Other:
- board size 251 x 101 mm -> 251 x 101.5 mm
