File: HT-manaita.kicad_sch (KiCad schematic)
At the start: 122 parts, among them J1 Conn_01x12_Pin, J2 Conn_01x12_Pin, SW1 SW_Push, SW10 SW_Push, SW11 SW_Push, SW12 SW_Push, SW13 SW_Push, SW14 SW_Push, SW15 SW_Push, SW16 SW_Push, SW17 SW_Push, SW18 SW_Push, SW19 SW_Push, SW2 SW_Push, SW20 SW_Push, SW21 SW_Push, SW22 SW_Push, SW23 SW_Push, SW24 SW_Push, SW25 SW_Push, SW26 SW_Push, SW27 SW_Push, SW28 SW_Push, SW29 SW_Push, SW3 SW_Push, SW30 SW_Push, SW31 SW_Push, SW32 SW_Push, SW33 SW_Push, SW34 SW_Push, SW35 SW_Push, SW36 SW_Push, SW37 SW_Push, SW38 SW_Push, SW39 SW_Push, SW4 SW_Push, SW40 SW_Push, SW41 SW_Push, SW42 SW_Push, SW43 SW_Push, SW44 SW_Push, SW45 SW_Push, SW46 SW_Push, SW47 SW_Push, SW48 SW_Push, SW49 SW_Push, SW5 SW_Push, SW50 SW_Push, SW51 SW_Push, SW52 SW_Push, SW53 SW_Push, SW54 SW_Push, SW55 SW_Push, SW56 SW_Push, SW57 SW_Push, SW58 SW_Push, SW59 SW_Push, SW6 SW_Push, SW60 SW_Push, SW7 SW_Push, SW8 SW_Push, SW9 SW_Push

Commit message: 部品配置・基板外形作成
Parts:
- removed SW19: SW_Push, Button_Switch_Keyboard:SW_Cherry_MX_1.00u_PCB, symbol Switch:SW_Push
Changed lines of the file:
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@@
   (junction (at 284.48 213.36) (diameter 0) (color 0 0 0 0)
   )
-  (junction (at 161.29 222.25) (diameter 0) (color 0 0 0 0)
-  )
   (junction (at 87.63 184.15) (diameter 0) (color 0 0 0 0)
   )
@@
     (stroke (width 0) (type default))
   )
-  (wire (pts (xy 161.29 203.2) (xy 161.29 222.25))
-    (stroke (width 0) (type default))
-  )
   (wire (pts (xy 345.44 184.15) (xy 345.44 203.2))
     (stroke (width 0) (type default))
@@
     (stroke (width 0) (type default))
   )
-  (wire (pts (xy 161.29 222.25) (xy 161.29 241.3))
+  (wire (pts (xy 161.29 203.2) (xy 161.29 241.3))
     (stroke (width 0) (type default))
   )
@@
         )
       )
-    )
-  )
-  (symbol (lib_id "Switch:SW_Push") (at 166.37 222.25 0) (unit 1)
-    (in_bom yes) (on_board yes) (dnp no) (fields_autoplaced)
-    (property "Reference" "SW19" (at 166.37 215.9 0)
-      (effects (font (size 1.27 1.27)))
-    )
-    (property "Value" "SW_Push" (at 166.37 218.44 0)
-      (effects (font (size 1.27 1.27)))
-    )
-    (property "Footprint" "Button_Switch_Keyboard:SW_Cherry_MX_1.00u_PCB" (at 166.37 217.17 0)
-      (effects (font (size 1.27 1.27)) hide)
-    )
-    (property "Datasheet" "~" (at 166.37 217.17 0)
-      (effects (font (size 1.27 1.27)) hide)
-    )
-    (pin "1")
-    (pin "2")
-    (instances
-      (project "HT-manaita"
-        (path "/e71272bd-3528-47c0-91cc-cb19803ae5f5"
-          (reference "SW19") (unit 1)
-        )
-      )

Commit message: HT-manaita_v1.0 基板作成
Connections:
- net COL0: no longer D1.1 (K), D10.1 (K), D11.1 (K), D13.1 (K), D14.1 (K), D15.1 (K), D16.1 (K), D17.1 (K), D19.1 (K), D2.1 (K), D20.1 (K), D21.1 (K), D22.1 (K), D23.1 (K), D25.1 (K), D26.1 (K), D27.1 (K), D28.1 (K), D29.1 (K), D3.1 (K), D32.2 (A), D33.2 (A), D34.2 (A), D35.2 (A), D36.2 (A), D38.2 (A), D39.2 (A), D4.1 (K), D40.2 (A), D41.2 (A), D42.2 (A), D44.2 (A), D45.2 (A), D46.2 (A), D47.2 (A), D48.2 (A), D50.2 (A), D51.2 (A), D52.2 (A), D53.2 (A), D54.2 (A), D57.2 (A), D58.2 (A), D59.2 (A), D60.2 (A), D7.1 (K), D8.1 (K), D9.1 (K), J1.10 (Pin_10), J1.11 (Pin_11), J1.8 (Pin_8), J1.9 (Pin_9)
- removed net GND: J1.3 (Pin_3), J1.4 (Pin_4), J2.2 (Pin_2)
- new net COL1: D10.1 (K), D11.1 (K), D17.1 (K), D23.1 (K), D29.1 (K), D35.2 (A), D36.2 (A), D4.1 (K), D42.2 (A), D48.2 (A), D54.2 (A), D60.2 (A), J1.11 (Pin_11)
- new net COL2: D15.1 (K), D16.1 (K), D22.1 (K), D28.1 (K), D3.1 (K), D34.2 (A), D40.2 (A), D41.2 (A), D47.2 (A), D53.2 (A), D59.2 (A), D9.1 (K), J1.10 (Pin_10)
- new net COL3: D14.1 (K), D2.1 (K), D20.1 (K), D21.1 (K), D27.1 (K), D33.2 (A), D39.2 (A), D45.2 (A), D46.2 (A), D52.2 (A), D58.2 (A), D8.1 (K), J1.9 (Pin_9)
- new net COL4: D1.1 (K), D13.1 (K), D19.1 (K), D25.1 (K), D26.1 (K), D32.2 (A), D38.2 (A), D44.2 (A), D50.2 (A), D51.2 (A), D57.2 (A), D7.1 (K), J1.8 (Pin_8)
- no-connect marks 17 -> 13

Commit message: v2.0 アップデート
Connections:
- net RW4 is gone; now on net ROW4: J2.12 (Pin_12)
- net COL0: now also SW1.1, SW2.1, SW3.1, SW31.1, SW32.1, SW33.1, SW34.1, SW35.1, SW4.1, SW5.1; no longer D12.1 (K), D18.1 (K), D24.1 (K), D30.1 (K), D31.2 (A), D37.2 (A), D43.2 (A), D49.2 (A), D5.1 (K), D55.2 (A), D56.2 (A), D6.1 (K), J1.7 (Pin_7)
- net COL1: now also SW10.1, SW36.1, SW37.1, SW38.1, SW39.1, SW40.1, SW6.1, SW7.1, SW8.1, SW9.1; no longer D10.1 (K), D11.1 (K), D17.1 (K), D23.1 (K), D29.1 (K), D35.2 (A), D36.2 (A), D4.1 (K), D42.2 (A), D48.2 (A), D54.2 (A), D60.2 (A)
- net COL2: now also SW11.1, SW12.1, SW13.1, SW14.1, SW15.1, SW41.1, SW42.1, SW43.1, SW44.1, SW45.1; no longer D15.1 (K), D16.1 (K), D22.1 (K), D28.1 (K), D3.1 (K), D34.2 (A), D40.2 (A), D41.2 (A), D47.2 (A), D53.2 (A), D59.2 (A), D9.1 (K)
- net COL3: now also SW16.1, SW17.1, SW18.1, SW20.1, SW46.1, SW47.1, SW48.1, SW49.1, SW50.1; no longer D14.1 (K), D2.1 (K), D20.1 (K), D21.1 (K), D27.1 (K), D33.2 (A), D39.2 (A), D45.2 (A), D46.2 (A), D52.2 (A), D58.2 (A), D8.1 (K)
- net COL4: now also SW21.1, SW22.1, SW23.1, SW24.1, SW25.1, SW51.1, SW52.1, SW53.1, SW54.1, SW55.1; no longer D1.1 (K), D13.1 (K), D19.1 (K), D25.1 (K), D26.1 (K), D32.2 (A), D38.2 (A), D44.2 (A), D50.2 (A), D51.2 (A), D57.2 (A), D7.1 (K)
- net ROW0: now also D12.1 (K), D18.1 (K), D24.1 (K), D30.1 (K), D31.2 (A), D37.2 (A), D43.2 (A), D49.2 (A), D5.1 (K), D55.2 (A), D56.2 (A), D6.1 (K); no longer SW1.1, SW2.1, SW3.1, SW4.1, SW5.1
- net ROW1: now also D10.1 (K), D11.1 (K), D17.1 (K), D23.1 (K), D29.1 (K), D35.2 (A), D36.2 (A), D4.1 (K), D42.2 (A), D48.2 (A), D54.2 (A), D60.2 (A); no longer SW10.1, SW6.1, SW7.1, SW8.1, SW9.1
- net ROW2: now also D15.1 (K), D16.1 (K), D22.1 (K), D28.1 (K), D3.1 (K), D34.2 (A), D40.2 (A), D41.2 (A), D47.2 (A), D53.2 (A), D59.2 (A), D9.1 (K); no longer SW11.1, SW12.1, SW13.1, SW14.1, SW15.1
- net ROW3: now also D14.1 (K), D2.1 (K), D20.1 (K), D21.1 (K), D27.1 (K), D33.2 (A), D39.2 (A), D45.2 (A), D46.2 (A), D52.2 (A), D58.2 (A), D8.1 (K); no longer SW16.1, SW17.1, SW18.1, SW20.1
- net ROW4: now also D1.1 (K), D13.1 (K), D19.1 (K), D25.1 (K), D26.1 (K), D32.2 (A), D38.2 (A), D44.2 (A), D50.2 (A), D51.2 (A), D57.2 (A), D7.1 (K); no longer SW21.1, SW22.1, SW23.1, SW24.1, SW25.1
- net COL5: now reaches SW56.1, SW57.1, SW58.1, SW59.1, SW60.1
- net COL5: now also J1.7 (Pin_7), SW26.1, SW27.1, SW28.1, SW29.1, SW30.1
